File: board/nanook-as.kicad_pcb (KiCad board)
At the start: 2 copper layers, 46 x 28 mm, 14 parts, among them J1 Address, J2 Flow Ext, J3 Pressure Ext, J4 Pressure Int, U1 STM32F030F4Px, X1 I2C-6P, X2 SWD

Commit message: WIP
Parts:
- added C10: 100n, Capacitors_SMD:C_0805, F.Cu at (181.0, 117.0)
- added C11: 100n, Capacitors_SMD:C_0805, F.Cu at (180.5, 120.0)
- added C4: 10n, Capacitors_SMD:C_0805, F.Cu at (170.0, 118.0)
- added C5: 1u, Capacitors_SMD:C_0805, F.Cu at (169.5, 121.5)
- added C6: 100n, Capacitors_SMD:C_0805, F.Cu at (169.5, 124.5)
- added C7: 100n, Capacitors_SMD:C_0805, F.Cu at (175.5, 117.5)
- added C8: 100n, Capacitors_SMD:C_0805, F.Cu at (175.5, 121.0)
- added C9: 100n, Capacitors_SMD:C_0805, F.Cu at (175.5, 124.5)
- added J5: Conn_01x02, Connectors_JST:JST_XH_B02B-XH-A_02x2.50mm_Straight, F.Cu at (135.0, 93.0)
- added J6: Conn_01x02, Connectors_JST:JST_XH_B02B-XH-A_02x2.50mm_Straight, F.Cu at (132.0, 101.0)
- added J7: Conn_01x02, Connectors_JST:JST_XH_B02B-XH-A_02x2.50mm_Straight, F.Cu at (132.5, 108.5)
- added J8: Conn_01x02, Connectors_JST:JST_XH_B02B-XH-A_02x2.50mm_Straight, F.Cu at (125.0, 93.5)
- added L1: 22uH, Inductors_SMD:L_0805, F.Cu at (187.1, 106.0)
- added L2: 22uH, Inductors_SMD:L_0805, F.Cu at (187.1, 109.5)
- added L3: 22uH, Inductors_SMD:L_0805, F.Cu at (187.1, 113.5)
- added L4: 22uH, Inductors_SMD:L_0805, F.Cu at (187.1, 117.0)
- added L5: 22uH, Inductors_SMD:L_0805, F.Cu at (187.1, 120.5)
- added L6: 22uH, Inductors_SMD:L_0805, F.Cu at (187.1, 124.0)
- added L7: 22uH, Inductors_SMD:L_0805, F.Cu at (187.1, 127.5)
- added R5: 100k, Resistors_SMD:R_0805, F.Cu at (135.5, 124.5)
- added R6: 100k, Resistors_SMD:R_0805, F.Cu at (135.0, 128.0)
- added R7: 100k, Resistors_SMD:R_0805, F.Cu at (134.9, 132.0)
- added R8: 100k, Resistors_SMD:R_0805, F.Cu at (134.5, 135.5)
- added U2: SPX3819, TO_SOT_Packages_SMD:SOT-23-5, F.Cu at (148.5, 105.0)
- J2: value Flow Ext -> Water Flow; footprint device.farm:DG301-5.0-03 -> Connectors_JST:JST_XH_B03B-XH-A_03x2.50mm_Straight
- J3: value Pressure Ext -> Conn_01x03; footprint device.farm:DG301-5.0-03 -> Connectors_JST:JST_XH_B03B-XH-A_03x2.50mm_Straight
- J4: value Pressure Int -> Conn_01x03; footprint device.farm:DG301-5.0-03 -> Connectors_JST:JST_XH_B03B-XH-A_03x2.50mm_Straight
- moved R2 39.2 mm to (130.6, 127.5), turned to 0 degrees
- moved R4 38.9 mm to (129.6, 135.0), turned to 0 degrees
- moved R1 36.8 mm to (131.1, 124.5), turned to 0 degrees
- moved R3 36.2 mm to (130.1, 131.5), turned to 0 degrees
- moved C2 35.2 mm to (164.5, 121.0), turned to 0 degrees
- moved C1 34.3 mm to (164.0, 118.0), turned to 0 degrees
- moved J2 32.4 mm to (166.0, 109.0)
- moved X2 30.4 mm to (138.0, 117.5)
- moved J1 29.7 mm to (180.0, 108.5), turned to 0 degrees
- moved C3 29.6 mm to (164.0, 124.5), turned to 0 degrees
- moved U1 25.6 mm to (150.5, 120.5)
- moved J3 17.6 mm to (166.0, 99.5)
- moved X1 16.7 mm to (148.3, 93.8)
- moved J4 13.1 mm to (165.5, 91.0)
Connections:
- C3 pad 1: +3V3 -> GND
- C3 pad 2: GND -> Net-(C3-Pad2)
- R1 pad 2: Net-(R1-Pad2) -> Net-(L2-Pad1)
- R2 pad 1: GND -> Net-(L2-Pad1)
- R2 pad 2: Net-(R1-Pad2) -> GND
- R3 pad 2: Net-(R3-Pad2) -> Net-(L3-Pad1)
- R4 pad 1: GND -> Net-(L3-Pad1)
- R4 pad 2: Net-(R3-Pad2) -> GND
- U1 pad 10: (no net) -> /Water Out/ADC-IN
- U1 pad 11: (no net) -> /Frigo In/ADC-IN
- U1 pad 12: (no net) -> /Frigo Out/ADC-IN
- U1 pad 14: (no net) -> Net-(J1-Pad2)
- U1 pad 5: +3V3 -> Net-(C3-Pad2)
- U1 pad 7: Net-(R1-Pad2) -> /Water Pressure/ADC-IN
- U1 pad 8: Net-(R3-Pad2) -> /Frigo Pressure/ADC-IN
- U1 pad 9: Net-(J1-Pad2) -> /Water In/ADC-IN
- X1 pad 4: +3V3 -> (no net)
Routing:
- net +5V: track 55.3 -> 0.00 mm, vias 1 -> 0
- net +3V3: track 46.0 -> 0.00 mm, vias 2 -> 0
- net Net-(J4-Pad2): track 42.9 -> 0.00 mm
- net GND: track 22.2 -> 0.00 mm, vias 5 -> 0
- net /ALERT: track 21.9 -> 0.00 mm, vias 2 -> 0
- net Net-(J3-Pad2): track 20.1 -> 0.00 mm
- net /SDA: track 18.6 -> 0.00 mm, vias 2 -> 0
- net Net-(R1-Pad2): track 16.6 -> 0.00 mm, vias 2 -> 0
- net Net-(J1-Pad2): track 15.6 -> 0.00 mm, vias 2 -> 0
- net Net-(J2-Pad2): track 15.4 -> 0.00 mm
- net /SCL: track 12.4 -> 0.00 mm, vias 2 -> 0
- net Net-(C1-Pad1): track 9.10 -> 0.00 mm, vias 2 -> 0
- net /SWDIO: track 7.03 -> 0.00 mm
- net Net-(R3-Pad2): track 5.58 -> 0.00 mm
- net /SWCLK: track 3.24 -> 0.00 mm
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- removed copper zone on B.Cu, net GND
Other:
- board outline removed
- board text removed: "5V"
- board text removed: "COLD"
- board text removed: "GND"
- board text removed: "HOT"
- board text removed: "IAS3A v1.0"
- board text removed: "REFRIGERANT PRESSURE"
- board text removed: "SGN"
- board text removed: "SIDE"
- board text removed: "WATER FLOW"
- board text removed: "WATER PRESSURE"

Commit message: WIP
Parts:
- J2, J3, J4: footprint Connectors_JST:JST_XH_B03B-XH-A_03x2.50mm_Straight -> Connectors_JST:JST_XH_S03B-XH-A_03x2.50mm_Angled
- J5, J6, J7, J8: footprint Connectors_JST:JST_XH_B02B-XH-A_02x2.50mm_Straight -> Connectors_JST:JST_XH_S02B-XH-A_02x2.50mm_Angled
- moved J8 86.7 mm to (209.5, 113.0)
- moved R8 80.6 mm to (209.5, 106.0)
- moved X2 70.2 mm to (203.0, 91.0)
- moved R7 70.1 mm to (200.0, 106.0)
- moved J7 67.6 mm to (200.0, 113.0)
- moved J6 59.7 mm to (190.5, 113.0)
- moved R6 59.7 mm to (190.5, 106.0)
- moved R4 53.1 mm to (174.0, 106.0)
- moved J5 50.2 mm to (181.0, 113.0)
- moved R5 49.1 mm to (181.0, 106.0)
- moved R3 46.6 mm to (169.0, 106.0)
- moved U1 44.9 mm to (186.0, 93.0)
- moved C2 40.7 mm to (193.0, 92.0)
- moved R2 38.1 mm to (162.0, 106.0)
- moved C11 36.7 mm to (213.5, 104.0), turned to 270 degrees
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Routing:
- net +3V3: track 0.00 -> 133.4 mm
- net +5V: track 0.00 -> 58.7 mm
- net /SCL: track 0.00 -> 58.4 mm, vias 0 -> 2
- net Net-(J2-Pad2): track 0.00 -> 54.3 mm, vias 0 -> 4
- net /SDA: track 0.00 -> 50.5 mm, vias 0 -> 2
- net /ALERT: track 0.00 -> 49.8 mm, vias 0 -> 4
- net GND: track 0.00 -> 47.6 mm, vias 0 -> 15
- net /Water Pressure/ADC-IN: track 0.00 -> 33.5 mm, vias 0 -> 2
- net /Frigo Out/ADC-IN: track 0.00 -> 27.9 mm
- net /SWCLK: track 0.00 -> 20.7 mm, vias 0 -> 1
- net /Frigo In/ADC-IN: track 0.00 -> 18.5 mm
- net /Frigo Pressure/ADC-IN: track 0.00 -> 18.3 mm
- net /Water Out/ADC-IN: track 0.00 -> 15.3 mm
- net /SWDIO: track 0.00 -> 15.1 mm, vias 0 -> 1
- net /Water In/ADC-IN: track 0.00 -> 12.1 mm
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- added copper zone on B.Cu, net GND
Other:
- board outline added: 75 x 42 mm
- board text added: "COLD"
- board text added: "FRIGO IN"
- board text added: "FRIGO OUT"
- board text added: "FRIGO PRESSURE"
- board text added: "HOT"
- board text added: "I2C"
- board text added: "NANOOK-AS v1.0"
- board text added: "SWD"
- board text added: "WATER FLOW"
- board text added: "WATER IN"
- board text added: "WATER OUT"
- board text added: "WATER PRESSURE"

Commit message: WIP
Parts:
- C1, C10, C11, C2, C3, C4, C5, C6, C7, C8, C9: footprint Capacitors_SMD:C_0805 -> Capacitor_SMD:C_0805_2012Metric
- J1: footprint Connectors:GS3 -> Jumper:SolderJumper-3_P1.3mm_Open_Pad1.0x1.5mm
- J2, J3, J4: footprint Connectors_JST:JST_XH_S03B-XH-A_03x2.50mm_Angled -> Connector_JST:JST_XH_S3B-XH-A-1_1x03_P2.50mm_Horizontal
- J5, J6, J7, J8: footprint Connectors_JST:JST_XH_S02B-XH-A_02x2.50mm_Angled -> Connector_JST:JST_XH_S2B-XH-A-1_1x02_P2.50mm_Horizontal
- L1, L2, L3, L4, L5, L6, L7: footprint Inductors_SMD:L_0805 -> Inductor_SMD:L_0805_2012Metric
- R1, R2, R3, R4, R5, R6, R7, R8: footprint Resistors_SMD:R_0805 -> Resistor_SMD:R_0805_2012Metric
- U1: footprint Housings_SSOP:TSSOP-20_4.4x6.5mm_Pitch0.65mm -> Package_SO:TSSOP-20_4.4x6.5mm_P0.65mm
- U2: footprint TO_SOT_Packages_SMD:SOT-23-5 -> Package_TO_SOT_SMD:SOT-23-5
- turned J1 to 90 degrees
Connections:
- U1 pad 2: (no net) -> Net-(U1-Pad2)
- U1 pad 3: (no net) -> Net-(U1-Pad3)
- X1 pad 4: (no net) -> Net-(X1-Pad4)
