File: board/nanook-as.kicad_pcb (KiCad board)
At the start: 2 copper layers, 75 x 42 mm, 38 parts, among them J1 Address, J2 Water Flow, J3 Conn_01x03, J4 Conn_01x03, J5 Conn_01x02, J6 Conn_01x02, J7 Conn_01x02, J8 Conn_01x02, U1 STM32F030F4Px, U2 SPX3819, X1 I2C-6P, X2 SWD

Commit message: WIP
Parts:
- R5, R6, R7, R8: value 100k -> (README.md)
- renumbered C5 to C1, C4 to C2, C2 to C3, C3 to C4, C1 to C5, J2 to J1, J1 to J2, U2 to U1, U1 to U2
Connections:
- U2 pad 2: Net-(U1-Pad2) -> unconnected-(U2-PF0)
- U2 pad 3: Net-(U1-Pad3) -> unconnected-(U2-PF1)
- X1 pad 4: Net-(X1-Pad4) -> unconnected-(X1-3V3)
Other:
- net class Default removed
- net class PWR removed

Commit message: WIP
Parts:
- removed the C1 at (161.0, 92.0)
- removed X2: SWD, device.farm:SWD
- added C10: 100n, Capacitor_SMD:C_0805_2012Metric, F.Cu at (231.0, 101.7)
- added C11: 100n, Capacitor_SMD:C_0805_2012Metric, F.Cu at (231.0, 104.7)
- added C3: 15p, Capacitor_SMD:C_0805_2012Metric, F.Cu at (226.6, 95.7)
- added C6: 100n, Capacitor_SMD:C_0805_2012Metric, F.Cu at (226.6, 104.7)
- added C7: 100n, Capacitor_SMD:C_0805_2012Metric, F.Cu at (231.0, 92.7)
- added C8: 100n, Capacitor_SMD:C_0805_2012Metric, F.Cu at (231.0, 95.7)
- added C9: 100n, Capacitor_SMD:C_0805_2012Metric, F.Cu at (231.0, 98.7)
- added J3: USB, Connector_PinHeader_2.54mm:PinHeader_1x03_P2.54mm_Vertical, F.Cu at (235.6, 104.9)
- added L2: 22uH, Inductor_SMD:L_0805_2012Metric, F.Cu at (244.0, 101.2)
- added NT1: NetTie_2, NetTie:NetTie-2_THT_Pad0.3mm, F.Cu at (238.7, 110.6)
- added NT2: NetTie_2, NetTie:NetTie-2_THT_Pad0.3mm, F.Cu at (239.0, 112.0)
- added R1: 10k, Resistor_SMD:R_0805_2012Metric, F.Cu at (243.9, 92.6)
- added R2: 10k, Resistor_SMD:R_0805_2012Metric, F.Cu at (243.9, 95.6)
- added Y1: 40MHz, Crystal:Crystal_SMD_3225-4Pin_3.2x2.5mm_HandSoldering, F.Cu at (227.7, 109.0)
- C2: value 10n -> 1u
- C4: value 100n -> 15p
- U1: value SPX3819 -> CD4051B; footprint Package_TO_SOT_SMD:SOT-23-5 -> Package_SO:SOIC-16_3.9x9.9mm_P1.27mm
- U2: value STM32F030F4Px -> ESP32-C3FN4; footprint Package_SO:TSSOP-20_4.4x6.5mm_P0.65mm -> Package_DFN_QFN:QFN-32-1EP_5x5mm_P0.5mm_EP3.45x3.45mm
- X1: footprint device.farm:Micro-Match-FOB-6 -> Drake:Micro-Match-FOB-6
- moved U1 80.6 mm to (237.5, 96.9)
- moved C2 66.7 mm to (226.6, 92.7), turned to 0 degrees
- moved L1 66.2 mm to (244.0, 98.4)
- moved U2 57.1 mm to (241.6, 106.2)
- moved C5 50.0 mm to (226.6, 101.7), turned to 0 degrees
- moved C4 48.7 mm to (226.6, 98.7)
- moved C1 34.2 mm to (227.0, 88.0)
- moved J2 26.1 mm to (222.0, 90.0)
- renumbered C3 to C1, C6 to C12, C7 to C13, C8 to C14, C9 to C15, C10 to C16, C11 to C17, J3 to J4, J4 to J5, J5 to J6, J6 to J7, J7 to J8, J8 to J9, L2 to L3, L3 to L4, L4 to L5, L5 to L6, L6 to L7, L7 to L8, R8 to R10, R1 to R3, R2 to R4, R3 to R5, R4 to R6, R5 to R7, R6 to R8, R7 to R9
Connections:
- C1 pad 2: GND -> +3V3
- C12 pad 1: /Water Pressure/ADC-IN -> /WATER_PRESSURE
- C13 pad 1: /Frigo Pressure/ADC-IN -> /FRIGO_PRESSURE
- C14 pad 1: /Water In/ADC-IN -> /WATER_IN
- C15 pad 1: /Water Out/ADC-IN -> /WATER_OUT
- C16 pad 1: /Frigo In/ADC-IN -> /FRIGO_IN
- C17 pad 1: /Frigo Out/ADC-IN -> /FRIGO_OUT
- C2 pad 1: GND -> Net-(U2-CHIP_EN)
- C2 pad 2: Net-(U1-BP) -> GND
- C4 pad 2: Net-(U2-VDDA) -> Net-(U2-XTAL_P)
- C5 pad 1: Net-(U2-NRST) -> /ADC
- J1 pad 2: Net-(J1-Pin_2) -> /WATER_FLOW
- J1 pad 3: +5V -> +5VA
- J2 pad 2: Net-(J2-C) -> /I2C_ADDR
- J4 pad 3: +5V -> +5VA
- J5 pad 3: +5V -> +5VA
- J6 pad 2: +3V3 -> +3.3VA
- J7 pad 2: +3V3 -> +3.3VA
- J8 pad 2: +3V3 -> +3.3VA
- J9 pad 2: +3V3 -> +3.3VA
- L1 pad 1: +3V3 -> Net-(L1-Pad1)
- L1 pad 2: Net-(U2-VDDA) -> +5VA
- L3 pad 2: /Water Pressure/ADC-IN -> /WATER_PRESSURE
- L4 pad 2: /Frigo Pressure/ADC-IN -> /FRIGO_PRESSURE
- L5 pad 2: /Water In/ADC-IN -> /WATER_IN
- L6 pad 2: /Water Out/ADC-IN -> /WATER_OUT
- L7 pad 2: /Frigo In/ADC-IN -> /FRIGO_IN
- L8 pad 2: /Frigo Out/ADC-IN -> /FRIGO_OUT
- U1 pad 1: +5V -> /WATER_OUT
- U1 pad 2: GND -> /FRIGO_OUT
- U1 pad 3: +5V -> /ADC
- U1 pad 4: Net-(U1-BP) -> GND
- U1 pad 5: +3V3 -> /FRIGO_IN
- U2 pad 1: GND -> unconnected-(U2-LNA_IN)
- U2 pad 10: /Water Out/ADC-IN -> unconnected-(U2-MTDI/GPIO5/ADC2_CH0)
- U2 pad 11: /Frigo In/ADC-IN -> +3V3
- U2 pad 12: /Frigo Out/ADC-IN -> unconnected-(U2-MTCK/GPIO6)
- U2 pad 13: /ALERT -> unconnected-(U2-MTDO/GPIO7)
- U2 pad 14: Net-(J2-C) -> unconnected-(U2-GPIO8)
- U2 pad 15: GND -> unconnected-(U2-GPIO9/BOOT)
- U2 pad 16: +3V3 -> unconnected-(U2-GPIO10)
- U2 pad 17: /SCL -> +3V3
- U2 pad 18: /SDA -> unconnected-(U2-VDD_SPI/GPIO11)
- U2 pad 19: /SWDIO -> /SDA
- U2 pad 2: unconnected-(U2-PF0) -> +3V3
- U2 pad 20: /SWCLK -> /SCL
- U2 pad 3: unconnected-(U2-PF1) -> +3V3
- U2 pad 4: Net-(U2-NRST) -> /I2C_ADDR
- U2 pad 5: Net-(U2-VDDA) -> unconnected-(U2-XTAL_32K_N/ADC1_CH1)
- U2 pad 6: Net-(J1-Pin_2) -> Net-(U2-GPIO2/ADC1_CH2)
- U2 pad 7: /Water Pressure/ADC-IN -> Net-(U2-CHIP_EN)
- U2 pad 8: /Frigo Pressure/ADC-IN -> /ADC
- U2 pad 9: /Water In/ADC-IN -> unconnected-(U2-MTMS/GPIO4/ADC1_CH4)
Routing:
- net +3V3: track 133.4 -> 0.00 mm
- net +5V: track 58.7 -> 0.00 mm
- net /SCL: track 58.4 -> 0.00 mm, vias 2 -> 0
- net Net-(J1-Pin_2): track 54.3 -> 0.00 mm, vias 4 -> 0
- net +3.3VA: track 0.00 -> 52.9 mm
- net /SDA: track 50.5 -> 0.00 mm, vias 2 -> 0
- net /ALERT: track 49.8 -> 11.3 mm, vias 4 -> 1
- net /Water Pressure/ADC-IN: track 33.5 -> 0.00 mm, vias 2 -> 0
- net +5VA: track 0.00 -> 28.7 mm
- net /Frigo Out/ADC-IN: track 27.9 -> 0.00 mm
- net GND: track 47.6 -> 24.9 mm, vias 15 -> 7
- net /SWCLK: track 20.7 -> 0.00 mm, vias 1 -> 0
- net /WATER_FLOW: track 0.00 -> 18.9 mm, vias 0 -> 1
- net /Frigo In/ADC-IN: track 18.5 -> 0.00 mm
- net /Frigo Pressure/ADC-IN: track 18.3 -> 0.00 mm
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Other:
- board text removed: "SWD"

Commit message: WIP
Parts:
- removed the C6 at (226.6, 104.7)
- removed the C8 at (231.0, 95.7)
- removed L3, L4, L5, L6, L7, L8: 22uH, Inductor_SMD:L_0805_2012Metric
- moved L1 92.9 mm to (151.5, 107.5), turned to 180 degrees
- moved NT1 88.9 mm to (150.4, 99.8)
- moved U1 69.6 mm to (168.0, 94.0), turned to -90 degrees
- moved C1 55.3 mm to (173.0, 100.0), turned to 90 degrees
- moved R2 54.4 mm to (189.8, 90.8)
- moved R1 54.2 mm to (189.8, 93.2)
- moved U2 45.1 mm to (198.2, 94.0), turned to -90 degrees
- moved C5 41.2 mm to (186.2, 93.2), turned to -90 degrees
- moved J2 39.5 mm to (182.5, 89.8), turned to 0 degrees
- moved C8 38.8 mm to (193.0, 94.0), turned to -90 degrees
- moved NT2 38.8 mm to (208.2, 88.5)
- moved C9 38.1 mm to (193.2, 100.0), turned to 180 degrees
- moved L2 37.0 mm to (208.8, 89.8), turned to -90 degrees
- moved C2 37.0 mm to (189.8, 95.8), turned to 180 degrees
- moved C7 28.3 mm to (204.2, 89.5)
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- renumbered C12 to C10, C13 to C11, C14 to C12, C15 to C13, C16 to C14, C17 to C15, C7 to C6, C9 to C7, C10 to C8, C11 to C9
Connections:
- C1 pad 1: +3V3 -> GND
- J6 pad 1: Net-(J6-Pin_1) -> /WATER_IN
- J7 pad 1: Net-(J7-Pin_1) -> /WATER_OUT
- J8 pad 1: Net-(J8-Pin_1) -> /FRIGO_IN
- J9 pad 1: Net-(J9-Pin_1) -> /FRIGO_OUT
- R10 pad 1: Net-(J9-Pin_1) -> /FRIGO_OUT
- R3 pad 2: Net-(L3-Pad1) -> /WATER_PRESSURE
- R4 pad 1: Net-(L3-Pad1) -> /WATER_PRESSURE
- R5 pad 2: Net-(L4-Pad1) -> /FRIGO_PRESSURE
- R6 pad 1: Net-(L4-Pad1) -> /FRIGO_PRESSURE
- R7 pad 1: Net-(J6-Pin_1) -> /WATER_IN
- R8 pad 1: Net-(J7-Pin_1) -> /WATER_OUT
- R9 pad 1: Net-(J8-Pin_1) -> /FRIGO_IN
- X1 pad 4: unconnected-(X1-3V3) -> +3V3
Routing:
- net /SCL: track 0.00 -> 57.3 mm, vias 0 -> 2
- net /SDA: track 0.00 -> 54.2 mm, vias 0 -> 2
- net /FRIGO_OUT: track 3.46 -> 54.0 mm
- net /FRIGO_IN: track 3.46 -> 46.6 mm, vias 0 -> 2
- net /A2: track 0.00 -> 42.4 mm, vias 0 -> 2
- net /A1: track 0.00 -> 42.1 mm, vias 0 -> 2
- net /A0: track 0.00 -> 41.9 mm, vias 0 -> 2
- net /ALERT: track 11.3 -> 52.8 mm, vias 1 -> 2
- net /ADC: track 0.00 -> 29.3 mm, vias 0 -> 2
- net /WATER_OUT: track 3.76 -> 32.6 mm
- net /WATER_IN: track 3.46 -> 31.4 mm
- net +3.3VA: track 52.9 -> 77.0 mm, vias 0 -> 3
- net +3V3: track 0.00 -> 21.7 mm, vias 0 -> 10
- net /WATER_PRESSURE: track 3.05 -> 23.4 mm
- net /USB+: track 0.00 -> 19.4 mm, vias 0 -> 1
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- added copper zone on B.Cu, net +3V3
- added copper zone on F.Cu, net GND
- removed copper zone on B.Cu, net GND
Other:
- board text added: "NANOOK-AS v1.1"
- board text removed: "NANOOK-AS v1.0"
