File: board/nanook-as.kicad_pcb (KiCad board)
At the start: 2 copper layers, 75 x 42 mm, 42 parts, among them J1 Water Flow, J2 Address, J3 USB, J4 Conn_01x03, J5 Conn_01x03, J6 Conn_01x02, J7 Conn_01x02, J8 Conn_01x02, J9 Conn_01x02, U1 CD4051B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

Commit message: WIP
Parts:
- Y1: footprint Crystal:Crystal_SMD_3225-4Pin_3.2x2.5mm_HandSoldering -> Crystal:Crystal_SMD_3225-4Pin_3.2x2.5mm
- moved C2 1.75 mm to (188.0, 95.8)
- moved C8 1.75 mm to (191.2, 94.0)
- moved R1 1.75 mm to (188.0, 93.2)
- moved R2 1.75 mm to (188.0, 90.8)
- moved C5 1.25 mm to (185.0, 93.2)
Connections:
- U1 pad 1: /WATER_OUT -> /FRIGO_IN
- U1 pad 12: /WATER_IN -> /WATER_OUT
- U1 pad 13: /WATER_FLOW -> /WATER_PRESSURE
- U1 pad 14: /WATER_PRESSURE -> /FRIGO_PRESSURE
- U1 pad 15: /FRIGO_PRESSURE -> /WATER_IN
- U1 pad 2: /FRIGO_OUT -> GND
- U1 pad 5: /FRIGO_IN -> /FRIGO_OUT
- U2 pad 10: unconnected-(U2-MTDI/GPIO5/ADC2_CH0-Pad10) -> /SDA
- U2 pad 12: unconnected-(U2-MTCK/GPIO6-Pad12) -> /ALERT
- U2 pad 13: unconnected-(U2-MTDO/GPIO7-Pad13) -> /WATER_FLOW
- U2 pad 14: unconnected-(U2-GPIO8-Pad14) -> /A0
- U2 pad 15: unconnected-(U2-GPIO9/BOOT-Pad15) -> /A1
- U2 pad 16: unconnected-(U2-GPIO10-Pad16) -> /A2
- U2 pad 19: /SDA -> unconnected-(U2-SPIHD/GPIO12-Pad19)
- U2 pad 20: /SCL -> unconnected-(U2-SPIWP/GPIO13-Pad20)
- U2 pad 21: /ALERT -> unconnected-(U2-SPICS0/GPIO14-Pad21)
- U2 pad 22: /A0 -> unconnected-(U2-SPICLK/GPIO15-Pad22)
- U2 pad 23: /A1 -> unconnected-(U2-SPID/GPIO16-Pad23)
- U2 pad 24: /A2 -> unconnected-(U2-SPIQ/GPIO17-Pad24)
- U2 pad 9: unconnected-(U2-MTMS/GPIO4/ADC1_CH4-Pad9) -> /SCL
Routing:
- net /WATER_FLOW: track 33.8 -> 57.7 mm, vias 0 -> 1
- net /A0: track 41.9 -> 34.0 mm
- net /A1: track 42.1 -> 34.7 mm
- net /WATER_IN: track 31.4 -> 24.3 mm
- net /A2: track 42.4 -> 36.4 mm
- net /FRIGO_IN: track 46.6 -> 41.0 mm, vias 2 -> 0
- net /WATER_OUT: track 32.6 -> 38.0 mm
- net /FRIGO_OUT: track 54.0 -> 58.3 mm, vias 0 -> 2
- net /ALERT: track 52.8 -> 48.8 mm
- net Net-(U2-CHIP_EN): track 11.5 -> 13.3 mm
- net Net-(U2-GPIO2/ADC1_CH2): track 8.44 -> 10.2 mm
- net +3V3: track 21.7 -> 23.5 mm
- net /SDA: track 54.2 -> 52.6 mm
- net /SCL: track 57.3 -> 58.6 mm
- net /ADC: track 29.3 -> 30.2 mm
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Other:
- board text added: "NANOOK-AS v1.2"
- board text removed: "NANOOK-AS v1.1"

Commit message: WIP
Parts:
- R10, R7, R8, R9: value (README.md) -> (cold: 4x 56k, hot: 3x 4k7 frigo in: 56k)
Changed lines of the file:
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@@
         (effects (font (size 1 1) (thickness 0.15)))
     )
-    (fp_text value "(README.md)" (at 0 1.65 90) (layer "F.Fab")
+    (fp_text value "(cold: 4x 56k, hot: 3x 4k7 frigo in: 56k)" (at 0 1.65 90) (layer "F.Fab")
         (effects (font (size 1 1) (thickness 0.15)))
     )
@@
         (effects (font (size 1 1) (thickness 0.15)))
     )
-    (fp_text value "(README.md)" (at 0 1.65 90) (layer "F.Fab")
+    (fp_text value "(cold: 4x 56k, hot: 3x 4k7 frigo in: 56k)" (at 0 1.65 90) (layer "F.Fab")
         (effects (font (size 1 1) (thickness 0.15)))
     )
@@
         (effects (font (size 1 1) (thickness 0.15)))
     )
-    (fp_text value "(README.md)" (at 0 1.65 90) (layer "F.Fab")
+    (fp_text value "(cold: 4x 56k, hot: 3x 4k7 frigo in: 56k)" (at 0 1.65 90) (layer "F.Fab")
         (effects (font (size 1 1) (thickness 0.15)))
     )
@@
         (effects (font (size 1 1) (thickness 0.15)))
     )
-    (fp_text value "(README.md)" (at 0 1.65 90) (layer "F.Fab")
+    (fp_text value "(cold: 4x 56k, hot: 3x 4k7 frigo in: 56k)" (at 0 1.65 90) (layer "F.Fab")
         (effects (font (size 1 1) (thickness 0.15)))
     )

Commit message: WIP
Parts:
- removed NT1, NT2: NetTie_2, NetTie:NetTie-2_THT_Pad0.3mm
- added C16: 10u, Capacitor_SMD:C_0805_2012Metric, F.Cu at (158.0, 98.0)
- added C17: 10u, Capacitor_SMD:C_0805_2012Metric, F.Cu at (152.0, 92.0)
- added L3: 22uH, Inductor_SMD:L_0805_2012Metric, F.Cu at (152.0, 89.5)
- added U3: LM1117MP-2.5, Package_TO_SOT_SMD:SOT-223-3_TabPin2, F.Cu at (158.0, 92.0)
- R10, R7, R8, R9: value (cold: 4x 56k, hot: 3x 4k7 frigo in: 56k) -> 4k7
- R3, R5: value 4k7 -> 10k
Connections:
- J6 pad 2: +3.3VA -> +2V5
- J7 pad 2: +3.3VA -> +2V5
- J8 pad 2: +3.3VA -> +2V5
- J9 pad 2: +3.3VA -> +2V5
- L1 pad 1: Net-(L1-Pad1) -> +5V
- L2 pad 1: Net-(L2-Pad1) -> +3V3
Routing:
- net +2V5: track 0.00 -> 116.3 mm, vias 0 -> 1
- net +3.3VA: track 77.0 -> 12.1 mm, vias 3 -> 2
- net +5V: track 0.00 -> 21.8 mm
- net Net-(U3-VO): track 0.00 -> 13.9 mm
- net Net-(L1-Pad1): track 8.51 -> 0.00 mm
- net +3V3: vias 10 -> 11
Other:
- board text added: "NANOOK-AS v1.3"
- board text removed: "NANOOK-AS v1.2"

Commit message: WIP
Parts:
- removed R2: 10k, Resistor_SMD:R_0805_2012Metric
Connections:
- U2 pad 6: Net-(U2-GPIO2/ADC1_CH2) -> unconnected-(U2-GPIO2/ADC1_CH2-Pad6)
Routing:
- net Net-(U2-GPIO2/ADC1_CH2): track 10.2 -> 0.00 mm
- net +3V3: vias 11 -> 10
