File: board/nanook-as.kicad_sch (KiCad schematic)
At the start: 12 parts

Commit message: WIP
Parts:
- removed ?: (no value), symbol Drake:SWD
- removed ? (x4): (no value), symbol Device:C
- removed ?: (no value), symbol MCU_ST_STM32F0:STM32F030F4Px
- removed ?: (no value), symbol Drake:SPX3819
- removed ?: (no value), symbol Device:L
- added C10, C11, C5, C6, C7, C8, C9: 100n, Capacitor_SMD:C_0805_2012Metric, symbol Device:C
- added C2: 1u, Capacitor_SMD:C_0805_2012Metric, symbol Device:C
- added C3, C4: 15p, Capacitor_SMD:C_0805_2012Metric, symbol Device:C
- added J3: USB, Connector_PinHeader_2.54mm:PinHeader_1x03_P2.54mm_Vertical, symbol Connector:Conn_01x03_Male
- added L2 (x2): 22uH, Inductor_SMD:L_0805_2012Metric, symbol Device:L
- added NT1, NT2: NetTie_2, NetTie:NetTie-2_THT_Pad0.3mm, symbol Device:NetTie_2
- added R2 (x2): 10k, Resistor_SMD:R_0805_2012Metric, symbol Device:R
- added U1: CD4051B, Package_SO:SOIC-16_3.9x9.9mm_P1.27mm, symbol Analog_Switch:CD4051B
- added U2: ESP32-C3FN4, Package_DFN_QFN:QFN-32-1EP_5x5mm_P0.5mm_EP3.45x3.45mm, symbol Espressif:ESP32-C3
- added Y1: 40MHz, Crystal:Crystal_SMD_3225-4Pin_3.2x2.5mm_HandSoldering, symbol Device:Crystal_GND24_Small
- C1: renamed from ?; value (none) -> 100n; footprint (none) -> Capacitor_SMD:C_0805_2012Metric
- J1: renamed from ?; value (none) -> Water Flow; footprint (none) -> Connector_JST:JST_XH_S3B-XH-A-1_1x03_P2.50mm_Horizontal
- J2: renamed from ?; value (none) -> Address; footprint (none) -> Jumper:SolderJumper-3_P1.3mm_Open_Pad1.0x1.5mm
- X1: renamed from ?; value (none) -> I2C-6P; footprint (none) -> Drake:Micro-Match-FOB-6
Connections:
- net +3V3: now also C1.2, C10.1, C11.1, C8.1, C9.1, NT2.1, R2.1, R2.1, U1.16 (VDD), U2.11 (VDD3P3_RTC), U2.17 (VDD3P3_CPU), U2.2 (VDD3P3), U2.3 (VDD3P3)
- net +5V: now also NT1.1; no longer J1.3 (Pin_3)
- net ALERT: now also U2.21 (SPICS0/GPIO14)
- net GND: now also C10.2, C11.2, C2.2, C3.1, C4.1, C5.2, C6.2, C7.2, C8.2, C9.2, J3.2 (Pin_2), U1.4 (X7), U1.6 (INH), U1.7 (VEE), U1.8 (VSS), U2.33 (GND), Y1.2, Y1.4; no longer C1.2
- net SCL: now also U2.20 (SPIWP/GPIO13)
- net SDA: now also U2.19 (SPIHD/GPIO12)
- net I2C_ADDR: now reaches J2.2 (C)
- net I2C_ADDR: now also U2.4 (XTAL_32K_P/ADC1_CH0)
- net WATER_FLOW: now reaches J1.2 (Pin_2)
- net WATER_FLOW: now also U1.13 (X0)
- new net: C2.1, R2.2, U2.7 (CHIP_EN)
- new net: L2.1, NT1.2
- new net: R2.2, U2.6 (GPIO2/ADC1_CH2)
- new net: L2.1, NT2.2
- new net: C4.2, U2.30 (XTAL_P), Y1.1
- new net: C3.2, U2.29 (XTAL_N), Y1.3
- new net +3.3VA: C6.1, C7.1, L2.2, U2.31 (VDDA), U2.32 (VDDA)
- new net +5VA: J1.3 (Pin_3), L2.2
- new net A0: U1.11 (A), U2.22 (SPICLK/GPIO15)
- new net A1: U1.10 (B), U2.23 (SPID/GPIO16)
- new net A2: U1.9 (C), U2.24 (SPIQ/GPIO17)
- new net ADC: C5.1, U1.3 (X), U2.8 (GPIO3/ADC1_CH3)
- new net FRIGO_IN: U1.5 (X5)
- new net FRIGO_OUT: U1.2 (X6)
- new net FRIGO_PRESSURE: U1.15 (X2)
- new net USB+: J3.1 (Pin_1), U2.26 (GPIO19/USB_D+)
- new net USB-: J3.3 (Pin_3), U2.25 (GPIO18/USB_D-)
- new net WATER_IN: U1.12 (X3)
- new net WATER_OUT: U1.1 (X4)
- new net WATER_PRESSURE: U1.14 (X1)
- no-connect marks 3 -> 13

Commit message: WIP
Parts:
- removed C6, C8: 100n, Capacitor_SMD:C_0805_2012Metric, symbol Device:C
- J3: symbol Connector:Conn_01x03_Male -> Connector_Generic:Conn_01x03
- renumbered C7 to C6, C9 to C7, C10 to C8, C11 to C9
Connections:
- net +3V3: now also X1.4 (3V3); no longer C1.1
- net GND: now also C1.1
- no-connect marks 13 -> 12
Other:
- moved on the sheet: J2, L2, NT1, NT2

Commit message: WIP
Parts:
- Y1: footprint Crystal:Crystal_SMD_3225-4Pin_3.2x2.5mm_HandSoldering -> Crystal:Crystal_SMD_3225-4Pin_3.2x2.5mm
Connections:
- net A0: now also U2.14 (GPIO8); no longer U2.22 (SPICLK/GPIO15)
- net A1: now also U2.15 (GPIO9/BOOT); no longer U2.23 (SPID/GPIO16)
- net A2: now also U2.16 (GPIO10); no longer U2.24 (SPIQ/GPIO17)
- net ALERT: now also U2.12 (MTCK/GPIO6); no longer U2.21 (SPICS0/GPIO14)
- net FRIGO_IN: now also U1.1 (X4); no longer U1.5 (X5)
- net FRIGO_OUT: now also U1.5 (X5); no longer U1.2 (X6)
- net FRIGO_PRESSURE: now also U1.14 (X1); no longer U1.15 (X2)
- net GND: now also U1.2 (X6)
- net SCL: now also U2.9 (MTMS/GPIO4/ADC1_CH4); no longer U2.20 (SPIWP/GPIO13)
- net SDA: now also U2.10 (MTDI/GPIO5/ADC2_CH0); no longer U2.19 (SPIHD/GPIO12)
- net WATER_FLOW: now also U2.13 (MTDO/GPIO7); no longer U1.13 (X0)
- net WATER_IN: now also U1.15 (X2); no longer U1.12 (X3)
- net WATER_OUT: now also U1.12 (X3); no longer U1.1 (X4)
- net WATER_PRESSURE: now also U1.13 (X0); no longer U1.14 (X1)
- no-connect marks 12 -> 11
Other:
- moved on the sheet: C1, C2, C3, C4, C5, C6, C7, C8, C9, J2, J3, L2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

Commit message: WIP
Parts:
- removed NT1, NT2: NetTie_2, NetTie:NetTie-2_THT_Pad0.3mm, symbol Device:NetTie_2
- added C16, C17: 10u, Capacitor_SMD:C_0805_2012Metric, symbol Device:C
- added L2: 22uH, Inductor_SMD:L_0805_2012Metric, symbol Device:L
- added U3: LM1117MP-2.5, Package_TO_SOT_SMD:SOT-223-3_TabPin2, symbol Regulator_Linear:LM1117MP-2.5
Connections:
- net +3V3: now also L2.1
- net +5V: now also L2.1, C16.1, U3.3 (VI)
- net GND: now also C16.2, C17.2, U3.1 (GND)
- new net: C17.1, L2.1, U3.2 (VO)
- new net +2V5: L2.2
Other:
- moved on the sheet: J2, L2

Commit message: WIP
Parts:
- removed R2: 10k, Resistor_SMD:R_0805_2012Metric, symbol Device:R
Connections:
- no-connect marks 11 -> 12
Changed lines of the file:
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@@
-(kicad_sch (version 20230221) (generator eeschema)
+(kicad_sch (version 20230409) (generator eeschema)
   (paper "A4")
   (junction (at 190.5 130.81) (diameter 0) (color 0 0 0 0)
@@
   (no_connect (at 88.9 41.91))
   (no_connect (at 144.78 31.75))
+  (no_connect (at 144.78 77.47))
   (no_connect (at 144.78 59.69))
   (no_connect (at 144.78 62.23))
@@
     (stroke (width 0) (type default))
   )
-  (wire (pts (xy 152.4 77.47) (xy 144.78 77.47))
-    (stroke (width 0) (type default))
-  )
   (wire (pts (xy 54.61 35.56) (xy 54.61 36.83))
     (stroke (width 0) (type default))
@@
         (path "/bd0055da-0838-4c4c-b506-87ee1119a3e6"
           (reference "#PWR0105") (unit 1)
-        )
-      )
-    )
-  )
-  (symbol (lib_id "Device:R") (at 156.21 77.47 270) (unit 1)
-    (in_bom yes) (on_board yes) (dnp no)
-    (property "Reference" "R2" (at 158.75 80.01 90)
-      (effects (font (size 1.27 1.27)))
-    )
-    (property "Value" "10k" (at 153.67 80.01 90)
-      (effects (font (size 1.27 1.27)))
-    )
-    (property "Footprint" "Resistor_SMD:R_0805_2012Metric" (at 156.21 75.692 90)
-      (effects (font (size 1.27 1.27)) hide)
-    )
-    (property "Datasheet" "~" (at 156.21 77.47 0)
-      (effects (font (size 1.27 1.27)) hide)
-    )
-    (pin "1")
-    (pin "2")
-    (instances
-      (project "nanook-as"
-        (path "/bd0055da-0838-4c4c-b506-87ee1119a3e6/00000000-0000-0000-0000-00005c22e635"
-          (reference "R2") (unit 1)
-        )
-        (path "/bd0055da-0838-4c4c-b506-87ee1119a3e6/00000000-0000-0000-0000-00005c22f26b"
-          (reference "R4") (unit 1)
-        )
-        (path "/bd0055da-0838-4c4c-b506-87ee1119a3e6"
-          (reference "R2") (unit 1)
         )
       )
@@
         )
       )
-    )
-  )
-  (symbol (lib_id "power:+3V3") (at 160.02 77.47 270) (unit 1)
-    (in_bom yes) (on_board yes) (dnp no)
-    (property "Reference" "#PWR0125" (at 156.21 77.47 0)
-      (effects (font (size 1.27 1.27)) hide)
-    )
-    (property "Value" "+3V3" (at 166.37 77.47 90)
-      (effects (font (size 1.27 1.27)))
-    )
-    (property "Footprint" "" (at 160.02 77.47 0)
-      (effects (font (size 1.27 1.27)) hide)
-    )
-    (property "Datasheet" "" (at 160.02 77.47 0)
-      (effects (font (size 1.27 1.27)) hide)
-    )
-    (pin "1")
-    (instances
-      (project "nanook-as"
-        (path "/bd0055da-0838-4c4c-b506-87ee1119a3e6"
-          (reference "#PWR0125") (unit 1)
-        )
-      )
