File: board/nanook-as.kicad_sch (KiCad schematic)
At the start: 12 parts

Commit message: WIP
Parts:
- removed ?: (no value), symbol Drake:SWD
- removed ? (x2): (no value), symbol Device:C
- removed ?: (no value), symbol MCU_ST_STM32F0:STM32F030F4Px
- removed ?: (no value), symbol Drake:SPX3819
- removed ?: (no value), symbol Device:L
- added H1 (x2): MountingHole, MountingHole:MountingHole_2.2mm_M2_Pad_Via, symbol Mechanical:MountingHole
- added J9: PROG, Connector_PinHeader_2.54mm:PinHeader_1x02_P2.54mm_Vertical, symbol Connector:Conn_01x02_Pin
- added U2: AMS1117-3.3, Package_TO_SOT_SMD:SOT-223-3_TabPin2, symbol Regulator_Linear:AMS1117-3.3
- added U3: ATtiny414-SS, Package_SO:SOIC-14_3.9x8.7mm_P1.27mm, symbol MCU_Microchip_ATtiny:ATtiny414-SS
- C1, C2: renamed from ?; value (none) -> 10u; footprint (none) -> Capacitor_SMD:C_0805_2012Metric
- C3: renamed from ?; value (none) -> 100n; footprint (none) -> Capacitor_SMD:C_0805_2012Metric
- J1: renamed from ?; value (none) -> Water Flow; footprint (none) -> Connector_JST:JST_XH_S3B-XH-A-1_1x03_P2.50mm_Horizontal
- J2: renamed from ?; value (none) -> Address; footprint (none) -> Jumper:SolderJumper-3_P1.3mm_Open_Pad1.0x1.5mm
- X1: renamed from ?; value (none) -> I2C-6P; footprint (none) -> Drake:Micro-Match-FOB-6
Connections:
- net +3V3: now also C2.1, U2.2 (VO), U3.1 (VCC); no longer C1.2
- net +5V: now also C1.2, U2.3 (VI)
- net ALERT: now also U3.7 (PB2)
- net Frigo In/ADC-IN: now also U3.4 (PA6)
- net Frigo Out/ADC-IN: now also U3.5 (PA7)
- net Frigo Pressure/ADC-IN: now also U3.13 (PA3)
- net GND: now also C2.2, J9.1 (Pin_1), U2.1 (GND), U3.14 (GND); no longer C2.1
- net SCL: now also U3.9 (PB0)
- net SDA: now also U3.8 (PB1)
- net Water In/ADC-IN: now also U3.2 (PA4)
- net Water Out/ADC-IN: now also U3.3 (PA5)
- net Water Pressure/ADC-IN: now also U3.12 (PA2)
- net at J2.2 (C): now also U3.6 (PB3)
- net at J1.2 (Pin_2): now also U3.11 (PA1)
- new net ~{RESET}: J9.2 (Pin_2), U3.10 (~{RESET}/PA0)
- no-connect marks 3 -> 1
