File: board/pressure-sensor.kicad_sch (KiCad schematic)
At the start: 5 parts

Commit message: WIP
Parts:
- C12: renamed from ?; value (none) -> 100n; footprint (none) -> Capacitor_SMD:C_0805_2012Metric
- J4: renamed from ?; value (none) -> Conn_01x03; footprint (none) -> Connector_JST:JST_XH_S3B-XH-A-1_1x03_P2.50mm_Horizontal
- L3: renamed from ?; value (none) -> 22uH; footprint (none) -> Inductor_SMD:L_0805_2012Metric
- R3: renamed from ?; value (none) -> 4k7; footprint (none) -> Resistor_SMD:R_0805_2012Metric
- R4: renamed from ?; value (none) -> 10k; footprint (none) -> Resistor_SMD:R_0805_2012Metric
Connections:
- net +5V renamed +5VA

Commit message: WIP
Parts:
- removed L3: 22uH, Inductor_SMD:L_0805_2012Metric, symbol Device:L
- renumbered C12 to C10
Connections:
- net ADC-IN: now also R3.2, R4.1
Changed lines of the file:
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@@
-(kicad_sch (version 20221126) (generator eeschema)
+(kicad_sch (version 20221206) (generator eeschema)
   (paper "A4")
   (junction (at 116.84 76.2) (diameter 0) (color 0 0 0 0)
@@
     (stroke (width 0) (type default))
   )
-  (wire (pts (xy 128.27 76.2) (xy 130.81 76.2))
-    (stroke (width 0) (type default))
-  )
   (wire (pts (xy 102.87 68.58) (xy 116.84 68.58))
     (stroke (width 0) (type default))
   )
-  (wire (pts (xy 116.84 76.2) (xy 120.65 76.2))
+  (wire (pts (xy 116.84 76.2) (xy 130.81 76.2))
     (stroke (width 0) (type default))
   )
@@
   (symbol (lib_id "Device:C") (at 130.81 80.01 0) (unit 1)
     (in_bom yes) (on_board yes) (dnp no)
-    (property "Reference" "C12" (at 134.62 78.74 0)
+    (property "Reference" "C10" (at 134.62 78.74 0)
       (effects (font (size 1.27 1.27)) (justify left))
     )
@@
       (project "nanook-as"
         (path "/bd0055da-0838-4c4c-b506-87ee1119a3e6/00000000-0000-0000-0000-00005c22e635"
-          (reference "C12") (unit 1)
+          (reference "C10") (unit 1)
         )
         (path "/bd0055da-0838-4c4c-b506-87ee1119a3e6/00000000-0000-0000-0000-00005c22f26b"
-          (reference "C13") (unit 1)
+          (reference "C11") (unit 1)
         )
       )
-    )
-  )
-  (symbol (lib_id "Device:L") (at 124.46 76.2 90) (unit 1)
-    (in_bom yes) (on_board yes) (dnp no)
-    (property "Reference" "L3" (at 128.27 71.12 90)
-      (effects (font (size 1.27 1.27)))
-    )
-    (property "Value" "22uH" (at 128.27 73.66 90)
-      (effects (font (size 1.27 1.27)))
-    )
-    (property "Footprint" "Inductor_SMD:L_0805_2012Metric" (at 124.46 76.2 0)
-      (effects (font (size 1.27 1.27)) hide)
-    )
-    (property "Datasheet" "~" (at 124.46 76.2 0)
-      (effects (font (size 1.27 1.27)) hide)
-    )
-    (pin "1")
-    (pin "2")
-    (instances
-      (project "nanook-as"
-        (path "/bd0055da-0838-4c4c-b506-87ee1119a3e6/00000000-0000-0000-0000-00005c22e635"
-          (reference "L3") (unit 1)
-        )
-        (path "/bd0055da-0838-4c4c-b506-87ee1119a3e6/00000000-0000-0000-0000-00005c22f26b"
-          (reference "L4") (unit 1)
-        )
-      )

Commit message: WIP
Parts:
- R3: value 4k7 -> 10k
Changed lines of the file:
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@@
       (effects (font (size 1.27 1.27)))
     )
-    (property "Value" "4k7" (at 120.65 73.66 0)
+    (property "Value" "10k" (at 120.65 73.66 0)
       (effects (font (size 1.27 1.27)))
     )
