File: board/pressure-sensor.kicad_sch (KiCad schematic)
At the start: 5 parts

Commit message: WIP
Parts:
- C6: renamed from ?; value (none) -> 100n; footprint (none) -> Capacitor_SMD:C_0805_2012Metric
- J3: renamed from ?; value (none) -> Conn_01x03; footprint (none) -> Connector_JST:JST_XH_S3B-XH-A-1_1x03_P2.50mm_Horizontal
- L2: renamed from ?; value (none) -> 22uH; footprint (none) -> Inductor_SMD:L_0805_2012Metric
- R1: renamed from ?; value (none) -> 4k7; footprint (none) -> Resistor_SMD:R_0805_2012Metric
- R2: renamed from ?; value (none) -> 10k; footprint (none) -> Resistor_SMD:R_0805_2012Metric
