File: board/temp-sensor.kicad_sch (KiCad schematic)
At the start: 4 parts

Commit message: WIP
Parts:
- C14: renamed from ?; value (none) -> 100n; footprint (none) -> Capacitor_SMD:C_0805_2012Metric
- J6: renamed from ?; value (none) -> Conn_01x02; footprint (none) -> Connector_JST:JST_XH_S2B-XH-A-1_1x02_P2.50mm_Horizontal
- L5: renamed from ?; value (none) -> 22uH; footprint (none) -> Inductor_SMD:L_0805_2012Metric
- R7: renamed from ?; value (none) -> (README.md); footprint (none) -> Resistor_SMD:R_0805_2012Metric
Connections:
- net +3V3 renamed +3.3VA

Commit message: WIP
Parts:
- removed L5: 22uH, Inductor_SMD:L_0805_2012Metric, symbol Device:L
- renumbered C14 to C12
Connections:
- net ADC-IN: now also J6.1 (Pin_1), R7.1
Changed lines of the file:
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@@
-(kicad_sch (version 20221126) (generator eeschema)
+(kicad_sch (version 20221206) (generator eeschema)
   (paper "A4")
   (junction (at 139.7 72.39) (diameter 0) (color 0 0 0 0)
@@
     (stroke (width 0) (type default))
   )
-  (wire (pts (xy 152.4 72.39) (xy 156.21 72.39))
-    (stroke (width 0) (type default))
-  )
   (wire (pts (xy 127 72.39) (xy 139.7 72.39))
     (stroke (width 0) (type default))
   )
-  (wire (pts (xy 139.7 72.39) (xy 144.78 72.39))
+  (wire (pts (xy 139.7 72.39) (xy 156.21 72.39))
     (stroke (width 0) (type default))
   )
@@
     )
   )
-  (symbol (lib_id "Device:L") (at 148.59 72.39 90) (unit 1)
-    (in_bom yes) (on_board yes) (dnp no)
-    (property "Reference" "L5" (at 148.59 68.58 90)
-      (effects (font (size 1.27 1.27)))
-    )
-    (property "Value" "22uH" (at 148.59 70.485 90)
-      (effects (font (size 1.27 1.27)))
-    )
-    (property "Footprint" "Inductor_SMD:L_0805_2012Metric" (at 148.59 72.39 0)
-      (effects (font (size 1.27 1.27)) hide)
-    )
-    (property "Datasheet" "~" (at 148.59 72.39 0)
-      (effects (font (size 1.27 1.27)) hide)
-    )
-    (pin "1")
-    (pin "2")
-    (instances
-      (project "nanook-as"
-        (path "/bd0055da-0838-4c4c-b506-87ee1119a3e6/00000000-0000-0000-0000-00005c22fbc8"
-          (reference "L5") (unit 1)
-        )
-        (path "/bd0055da-0838-4c4c-b506-87ee1119a3e6/00000000-0000-0000-0000-00005c23178f"
-          (reference "L6") (unit 1)
-        )
-        (path "/bd0055da-0838-4c4c-b506-87ee1119a3e6/00000000-0000-0000-0000-00005c2318b8"
-          (reference "L7") (unit 1)
-        )
-        (path "/bd0055da-0838-4c4c-b506-87ee1119a3e6/00000000-0000-0000-0000-00005c2319d5"
-          (reference "L8") (unit 1)
-        )
-      )
-    )
-  )
   (symbol (lib_id "Device:C") (at 156.21 77.47 0) (unit 1)
     (in_bom yes) (on_board yes) (dnp no)
-    (property "Reference" "C14" (at 160.02 77.47 0)
+    (property "Reference" "C12" (at 160.02 77.47 0)
       (effects (font (size 1.27 1.27)) (justify left))
     )
@@
       (project "nanook-as"
         (path "/bd0055da-0838-4c4c-b506-87ee1119a3e6/00000000-0000-0000-0000-00005c22fbc8"
+          (reference "C12") (unit 1)
+        )
+        (path "/bd0055da-0838-4c4c-b506-87ee1119a3e6/00000000-0000-0000-0000-00005c23178f"
+          (reference "C13") (unit 1)
+        )
+        (path "/bd0055da-0838-4c4c-b506-87ee1119a3e6/00000000-0000-0000-0000-00005c2318b8"
           (reference "C14") (unit 1)
         )
-        (path "/bd0055da-0838-4c4c-b506-87ee1119a3e6/00000000-0000-0000-0000-00005c23178f"
+        (path "/bd0055da-0838-4c4c-b506-87ee1119a3e6/00000000-0000-0000-0000-00005c2319d5"
           (reference "C15") (unit 1)
         )
-        (path "/bd0055da-0838-4c4c-b506-87ee1119a3e6/00000000-0000-0000-0000-00005c2318b8"
-          (reference "C16") (unit 1)
-        )
-        (path "/bd0055da-0838-4c4c-b506-87ee1119a3e6/00000000-0000-0000-0000-00005c2319d5"
-          (reference "C17") (unit 1)
-        )
       )

Commit message: WIP
Parts:
- R7: value (README.md) -> (cold: 4x 56k, hot: 3x 4k7 frigo in: 56k)
Changed lines of the file:
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@@
-(kicad_sch (version 20230121) (generator eeschema)
+(kicad_sch (version 20230221) (generator eeschema)
   (paper "A4")
   (junction (at 139.7 72.39) (diameter 0) (color 0 0 0 0)
@@
       (effects (font (size 1.27 1.27)))
     )
-    (property "Value" "(README.md)" (at 144.78 78.74 0)
+    (property "Value" "(cold: 4x 56k, hot: 3x 4k7 frigo in: 56k)" (at 139.7 63.5 0)
       (effects (font (size 1.27 1.27)))
     )

Commit message: WIP
Parts:
- R7: value (cold: 4x 56k, hot: 3x 4k7 frigo in: 56k) -> 4k7
Connections:
- net +3.3VA renamed +2V5
Changed lines of the file:
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@@
       (effects (font (size 1.27 1.27)))
     )
-    (property "Value" "(cold: 4x 56k, hot: 3x 4k7 frigo in: 56k)" (at 139.7 63.5 0)
+    (property "Value" "4k7" (at 143.51 78.74 0)
       (effects (font (size 1.27 1.27)))
     )
@@
       (effects (font (size 1.27 1.27)) (justify left))
     )
-    (property "Value" "100n" (at 158.75 80.01 0)
+    (property "Value" "100n" (at 160.02 80.01 0)
       (effects (font (size 1.27 1.27)) (justify left))
     )
@@
         (path "/bd0055da-0838-4c4c-b506-87ee1119a3e6/00000000-0000-0000-0000-00005c2319d5"
           (reference "C15") (unit 1)
+        )
+      )
+    )
+  )
+  (symbol (lib_id "power:+2V5") (at 129.54 69.85 270) (unit 1)
+    (in_bom yes) (on_board yes) (dnp no) (fields_autoplaced)
+    (property "Reference" "#PWR09" (at 125.73 69.85 0)
+      (effects (font (size 1.27 1.27)) hide)
+    )
+    (property "Value" "+2V5" (at 132.715 70.1668 90)
+      (effects (font (size 1.27 1.27)) (justify left))
+    )
+    (property "Footprint" "" (at 129.54 69.85 0)
+      (effects (font (size 1.27 1.27)) hide)
+    )
+    (property "Datasheet" "" (at 129.54 69.85 0)
+      (effects (font (size 1.27 1.27)) hide)
+    )
+    (pin "1")
+    (instances
+      (project "nanook-as"
+        (path "/bd0055da-0838-4c4c-b506-87ee1119a3e6/00000000-0000-0000-0000-00005c22fbc8"
+          (reference "#PWR09") (unit 1)
+        )
+        (path "/bd0055da-0838-4c4c-b506-87ee1119a3e6/00000000-0000-0000-0000-00005c23178f"
+          (reference "#PWR010") (unit 1)
+        )
+        (path "/bd0055da-0838-4c4c-b506-87ee1119a3e6/00000000-0000-0000-0000-00005c2318b8"
+          (reference "#PWR011") (unit 1)
+        )
+        (path "/bd0055da-0838-4c4c-b506-87ee1119a3e6/00000000-0000-0000-0000-00005c2319d5"
+          (reference "#PWR012") (unit 1)
         )
       )
@@
         )
       )
-    )
-  )
-  (symbol (lib_id "power:+3.3VA") (at 129.54 69.85 270) (unit 1)
-    (in_bom yes) (on_board yes) (dnp no) (fields_autoplaced)
-    (property "Reference" "#PWR0137" (at 125.73 69.85 0)
-      (effects (font (size 1.27 1.27)) hide)
-    )
-    (property "Value" "+3.3VA" (at 132.715 70.1819 90)
-      (effects (font (size 1.27 1.27)) (justify left))
-    )
-    (property "Footprint" "" (at 129.54 69.85 0)
-      (effects (font (size 1.27 1.27)) hide)
-    )
-    (property "Datasheet" "" (at 129.54 69.85 0)
-      (effects (font (size 1.27 1.27)) hide)
-    )
-    (pin "1")
-    (instances
-      (project "nanook-as"
-        (path "/bd0055da-0838-4c4c-b506-87ee1119a3e6/00000000-0000-0000-0000-00005c22fbc8"
-          (reference "#PWR0137") (unit 1)
-        )
-        (path "/bd0055da-0838-4c4c-b506-87ee1119a3e6/00000000-0000-0000-0000-00005c23178f"
-          (reference "#PWR0140") (unit 1)
-        )
-        (path "/bd0055da-0838-4c4c-b506-87ee1119a3e6/00000000-0000-0000-0000-00005c2318b8"
-          (reference "#PWR0143") (unit 1)
-        )
-        (path "/bd0055da-0838-4c4c-b506-87ee1119a3e6/00000000-0000-0000-0000-00005c2319d5"
-          (reference "#PWR0146") (unit 1)
-        )
-      )
