File: board/temp-sensor.kicad_sch (KiCad schematic)
At the start: 4 parts

Commit message: WIP
Parts:
- C8: renamed from ?; value (none) -> 100n; footprint (none) -> Capacitor_SMD:C_0805_2012Metric
- J5: renamed from ?; value (none) -> Conn_01x02; footprint (none) -> Connector_JST:JST_XH_S2B-XH-A-1_1x02_P2.50mm_Horizontal
- L4: renamed from ?; value (none) -> 22uH; footprint (none) -> Inductor_SMD:L_0805_2012Metric
- R5: renamed from ?; value (none) -> (README.md); footprint (none) -> Resistor_SMD:R_0805_2012Metric
